Commit message: QtUWSim: updates to UWSim that allow ROSJointStateToArm interface receiving a full joint states vector including fixed and mimic joints. Added a ROS-compatible g500-ARM5 urdf file.

File: UWSim/data/scenes/g500ARM5-ros.urdf (robot description, URDF)
Before this commit: robot girona500, 8 links, 7 joints
Links:
- link base_link: geometry collision mesh filename=package://UWSim/data/robot/GIRONA500/g500_March11_collision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; visual mesh filename=package://UWSim/data/robot/GIRONA500/g500_March11.dae
- link part0: geometry collision mesh filename=package://UWSim/data/robot/ARM5E/ARM5E_part0_cs.dae; visual mesh filename=package://UWSim/data/robot/ARM5E/ARM5E_part0.dae
- link part1: geometry visual mesh filename=package://UWSim/data/robot/ARM5E/ARM5E_part1.dae
- link part2: geometry visual mesh filename=package://UWSim/data/robot/ARM5E/ARM5E_part2.dae
- link part3: geometry visual mesh filename=package://UWSim/data/robot/ARM5E/ARM5E_part3.dae
- link part4_base: geometry visual mesh filename=package://UWSim/data/robot/ARM5E/ARM5E_part4_base.dae
- link part4_jaw1: geometry visual mesh filename=package://UWSim/data/robot/ARM5E/ARM5E_part4_jaw1.dae
- link part4_jaw2: geometry visual mesh filename=package://UWSim/data/robot/ARM5E/ARM5E_part4_jaw2.dae
