Commit message: QtUWSim: multiple fixes in mosaic loading: auto-fitting, grasp specification with draggers, load geometry file directly without a scene, fixed some memory leaks (still more to fix\!)

File: UWSim/data/scenes/UNIBOHand.urdf (robot description, URDF)
Before this commit: robot UNIBOHand, 13 links, 12 joints
Joints:
- joint 1_finger_base_to_finger_slider: type continuous -> prismatic
- joint 2_finger_base_to_finger_slider: type continuous -> prismatic
- joint 3_finger_base_to_finger_slider: type continuous -> prismatic
