Commit message: preparing for release with bloom

File: UWSim/data/scenes/g500ARM5-rviz.urdf (robot description, URDF)
Before this commit: robot girona500, 8 links, 7 joints
Links:
- link base_link: geometry visual mesh filename=robot/GIRONA500/g500_March11.stl
- link part0: geometry visual mesh filename=robot/ARM5E/ARM5E_part0.dae
- link part1: geometry visual mesh filename=robot/ARM5E/ARM5E_part1.dae
- link part2: geometry visual mesh filename=robot/ARM5E/ARM5E_part2.dae
- link part3: geometry visual mesh filename=robot/ARM5E/ARM5E_part3.stl
- link part4_base: geometry visual mesh filename=robot/ARM5E/ARM5E_part4_base.dae
- link part4_jaw1: geometry visual mesh filename=robot/ARM5E/ARM5E_part4_jaw1.dae
- link part4_jaw2: geometry visual mesh filename=robot/ARM5E/ARM5E_part4_jaw2.dae

File: UWSim/data/scenes/g500ARM5.urdf (robot description, URDF)
Before this commit: robot girona500, 8 links, 7 joints
Links:
- link base_link: geometry visual mesh filename=robot/GIRONA500/g500_March11.osg
- link part0: geometry visual mesh filename=robot/ARM5E/ARM5E_part0.osg
- link part1: geometry visual mesh filename=robot/ARM5E/ARM5E_part1.osg
- link part2: geometry visual mesh filename=robot/ARM5E/ARM5E_part2.osg
- link part3: geometry visual mesh filename=robot/ARM5E/ARM5E_part3.osg
- link part4_base: geometry visual mesh filename=robot/ARM5E/ARM5E_part4_base.osg
- link part4_jaw1: geometry visual mesh filename=robot/ARM5E/ARM5E_part4_jaw1.osg
- link part4_jaw2: geometry visual mesh filename=robot/ARM5E/ARM5E_part4_jaw2.osg

File: UWSim/data/scenes/ujione-rviz.urdf (robot description, URDF)
Before this commit: robot girona500, 3 links, 2 joints
Links:
- link ujione_base: geometry visual mesh filename=robot/UJIOne/ujione_base.dae
- link ujione_jaw_inner: geometry visual mesh filename=robot/UJIOne/ujione_jaw_inner.dae
- link ujione_jaw_outer: geometry visual mesh filename=robot/UJIOne/ujione_jaw_outer.dae

File: UWSim/data/scenes/ujione.urdf (robot description, URDF)
Before this commit: robot girona500, 3 links, 2 joints
Links:
- link ujione_base: geometry visual mesh filename=robot/UJIOne/ujione_base.osg
- link ujione_jaw_inner: geometry visual mesh filename=robot/UJIOne/ujione_jaw_inner.osg
- link ujione_jaw_outer: geometry visual mesh filename=robot/UJIOne/ujione_jaw_outer.osg
