Commit message: UWSim now loads the file included on URDF instead of osg version. UWSim can load every file that osgviewer can open. Check you .urdf!

File: UWSim/data/scenes/g500ARM5.urdf (robot description, URDF)
Before this commit: robot girona500, 8 links, 7 joints
Links:
- link base_link: geometry visual mesh filename=package://UWSim/data/robot/GIRONA500/g500_March11.osg
- link part0: geometry visual mesh filename=package://UWSim/data/robot/ARM5E/ARM5E_part0.osg
- link part1: geometry visual mesh filename=package://UWSim/data/robot/ARM5E/ARM5E_part1.osg
- link part2: geometry visual mesh filename=package://UWSim/data/robot/ARM5E/ARM5E_part2.osg
- link part3: geometry visual mesh filename=package://UWSim/data/robot/ARM5E/ARM5E_part3.osg
- link part4_base: geometry visual mesh filename=package://UWSim/data/robot/ARM5E/ARM5E_part4_base.osg
- link part4_jaw1: geometry visual mesh filename=package://UWSim/data/robot/ARM5E/ARM5E_part4_jaw1.osg
- link part4_jaw2: geometry visual mesh filename=package://UWSim/data/robot/ARM5E/ARM5E_part4_jaw2.osg

Commit message: UWSim: merge of r205 into trunk, use of resource_retriever for loading resources

File: UWSim/data/scenes/g500ARM5.urdf (robot description, URDF)
Before this commit: robot girona500, 8 links, 7 joints
Links:
- link base_link: geometry collision mesh filename=package://UWSim/data/robot/GIRONA500/g500_March11_collision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; visual mesh filename=package://UWSim/data/robot/GIRONA500/g500_March11.osg
- link part0: geometry collision mesh filename=package://UWSim/data/robot/ARM5E/ARM5E_part0_cs.osg; visual mesh filename=package://UWSim/data/robot/ARM5E/ARM5E_part0.osg

Commit message: Merged benchmark branch changes on UWSim into trunk,

File: UWSim/data/scenes/g500ARM5.urdf (robot description, URDF)
Before this commit: robot girona500, 8 links, 7 joints
Links:
- link base_link: geometry visual mesh filename=package://UWSim/data/robot/GIRONA500/g500_March11.osg
- link part0: geometry visual mesh filename=package://UWSim/data/robot/ARM5E/ARM5E_part0.osg

Commit message: preparing for release with bloom

File: UWSim/data/scenes/g500ARM5.urdf (robot description, URDF)
Before this commit: robot girona500, 8 links, 7 joints
Links:
- link base_link: geometry visual mesh filename=robot/GIRONA500/g500_March11.osg
- link part0: geometry visual mesh filename=robot/ARM5E/ARM5E_part0.osg
- link part1: geometry visual mesh filename=robot/ARM5E/ARM5E_part1.osg
- link part2: geometry visual mesh filename=robot/ARM5E/ARM5E_part2.osg
- link part3: geometry visual mesh filename=robot/ARM5E/ARM5E_part3.osg
- link part4_base: geometry visual mesh filename=robot/ARM5E/ARM5E_part4_base.osg
- link part4_jaw1: geometry visual mesh filename=robot/ARM5E/ARM5E_part4_jaw1.osg
- link part4_jaw2: geometry visual mesh filename=robot/ARM5E/ARM5E_part4_jaw2.osg

Commit message: Now ROStoArmJoint respect names given on messages independently from order. Changed urdf names to make them more user-friendly Updated interface examples

File: UWSim/data/scenes/g500ARM5.urdf (robot description, URDF)
Before this commit: robot girona500, 8 links, 7 joints
Joints:
- removed joint part0_to_part1
- removed joint part1_to_part2
- removed joint part2_to_part3
- removed joint part3_to_part4_base
- removed joint part4_to_part4_jaw1
- added joint Elbow: type continuous, parent part2, child part3, origin xyz=0.44278 0 0 rpy= 0 0.262 0 , axis 0 1 0
- added joint JawOpening: type continuous, parent part4_base, child part4_jaw1, origin xyz=0.07 0 0.04 rpy=0 0 0, axis 0 -1 0
- added joint JawRotate: type continuous, parent part3, child part4_base, origin xyz=0.320 0 0.077  rpy=0 0 0, axis 1 0 0
- added joint Shoulder: type continuous, parent part1, child part2, origin xyz=0.077 0 -0.130 rpy=0 0.209 0, axis 0 1 0
- added joint Slew: type continuous, parent part0, child part1, origin xyz=0 0 0 rpy=0 0 0, axis 0 0 -1

Commit message: Changed angular/linear factor to constraints supporting limits Fixed error on g500ARM5.urdf

File: UWSim/data/scenes/g500ARM5.urdf (robot description, URDF)
Before this commit: robot girona500, 8 links, 7 joints
Joints:
- joint part4_to_part4_jaw2: mimic joint=part4_to_part4_jaw1 multiplier=1 offset=0 -> joint=JawOpening multiplier=1 offset=0
