Commit message: Fixed bug with g500ARM5_laser.urdf joints names

File: UWSim/data/scenes/g500ARM5_laser.urdf (robot description, URDF)
Before this commit: robot girona500, 9 links, 8 joints
Joints:
- removed joint part0_to_part1
- removed joint part1_to_part2
- removed joint part2_to_part3
- removed joint part3_to_part4_base
- removed joint part4_to_part4_jaw1
- added joint Elbow: type continuous, parent part2, child part3, origin xyz=0.44278 0 0 rpy= 0 0.262 0 , axis 0 1 0
- added joint JawOpening: type continuous, parent part4_base, child part4_jaw1, origin xyz=0.07 0 0.04 rpy=0 -1 0, axis 0 -1 0
- added joint JawRotate: type continuous, parent part3, child part4_base, origin xyz=0.320 0 0.077  rpy=1.57 0 0, axis 1 0 0
- added joint Shoulder: type continuous, parent part1, child part2, origin xyz=0.077 0 -0.130 rpy=0 0.209 0, axis 0 1 0
- added joint Slew: type continuous, parent part0, child part1, origin xyz=0 0 0 rpy=0 0 0, axis 0 0 -1
- joint part4_to_part4_jaw2: mimic joint=part4_to_part4_jaw1 multiplier=1 offset=0 -> joint=JawOpening multiplier=1 offset=0
