Commit message: Fixed old references to UWSim package on cirs_sls scene

File: uwsim/data/scenes/g500ARM5_laser.urdf (robot description, URDF)
Before this commit: robot girona500, 9 links, 8 joints
Links:
- link base_link: geometry visual mesh filename=robot/GIRONA500/g500_March11.osg
- link part0: geometry visual mesh filename=robot/ARM5E/ARM5E_part0.osg
- link part1: geometry visual mesh filename=robot/ARM5E/ARM5E_part1.osg
- link part2: geometry visual mesh filename=robot/ARM5E/ARM5E_part2.osg
- link part3: geometry visual mesh filename=robot/ARM5E/ARM5E_part3.osg
- link part4_base: geometry visual mesh filename=robot/ARM5E/ARM5E_part4_base.osg
- link part4_jaw1: geometry visual mesh filename=robot/ARM5E/ARM5E_part4_jaw1long.osg
- link part4_jaw2: geometry visual mesh filename=robot/ARM5E/ARM5E_part4_jaw2long.osg

Commit message: fixed sls scene and model

File: uwsim/data/scenes/g500ARM5_laser.urdf (robot description, URDF)
Before this commit: robot girona500, 9 links, 8 joints
Links:
- link base_link: mass None -> 95
- link part4_jaw1: geometry visual mesh filename=robot/ARM5E/ARM5E_part4_jaw1.osg
- link part4_jaw2: geometry visual mesh filename=robot/ARM5E/ARM5E_part4_jaw2.osg
Joints:
- removed joint part3_to_sls
- added joint sls_to_part0: type fixed, parent part0, child sls, origin xyz=-0.5 0.1 0 rpy=3.1416 0 1.57
- joint JawOpening: origin xyz=0.07 0 0.04 rpy=0 -1 0 -> xyz=0.07 0 0.04 rpy=0 0 0
- joint JawRotate: origin xyz=0.320 0 0.077  rpy=1.57 0 0 -> xyz=0.320 0 0.077  rpy=0 0 0
- joint part4_to_part4_jaw2: origin xyz=0.07 0 -0.04 rpy=0 1 0 -> xyz=0.07 0 -0.04 rpy=0 0 0

Commit message: relative references to useful components and added frames to tf publishing

File: uwsim/data/scenes/g500ARM5_laser.urdf (robot description, URDF)
Before this commit: robot girona500, 9 links, 8 joints
Links:
- added link stereo_down_optical
Joints:
- added joint stereo_down_optical_to_part0: type fixed, parent part0, child stereo_down_optical, origin xyz=-0.5 -0.06 0 rpy=3.1416 0 1.57
