Commit message: New urdf based on the DH model of the ARM5E. Xacro based.

File: uwsim/data/scenes/g500ARM5.urdf (robot description, URDF)
Before this commit: robot girona500, 8 links, 7 joints
Links:
- added link end_effector
- added link kinematic_base
Joints:
- removed joint part4_to_part4_jaw2
- added joint part0_to_kinematic_base: type fixed, parent part0, child kinematic_base, origin xyz=0 0 0.13 rpy=0 0 0
- added joint part4_base_to_end_effector: type fixed, parent part4_base, child end_effector, origin xyz=0 0 0.1485 rpy=0 0 0
- added joint part4_to_link4_jaw2: type continuous, parent part4_base, child part4_jaw2, origin xyz=0.04 0 0.0450 rpy=0 0 0, axis 0 1 0, mimic joint=JawOpening multiplier=1 offset=0
- joint Elbow: axis 0 1 0 -> 0 0 1; limit (none) -> lower=0 upper=2.15294 effort=1000.0 velocity=1.0; origin xyz=0.44278 0 0 rpy= 0 0.262 0  -> xyz=0.438492379277 0.0614700067987 0 rpy=0 0 0.139277274
- joint JawOpening: limit (none) -> lower=-0.05816 upper=1.337696 effort=1000.0 velocity=1.0; origin xyz=0.07 0 0.04 rpy=0 0 0 -> xyz=-0.04 0 0.045 rpy=0 0 0
- joint JawRotate: axis 1 0 0 -> 0 0 1; origin xyz=0.320 0 0.077  rpy=0 0 0 -> xyz=0.349117258152 0.058023572508 0 rpy=1.570796327 0 1.972222055
- joint Shoulder: axis 0 1 0 -> 0 0 1; limit (none) -> lower=0 upper=1.58665 effort=1000.0 velocity=1.0; origin xyz=0.077 0 -0.130 rpy=0 0.209 0 -> xyz=0.08052 0 0 rpy=1.570796327 0 0
- joint Slew: axis 0 0 -1 -> 0 0 1; limit (none) -> lower=-1.570796327 upper=0.5488 effort=1000.0 velocity=1.0; parent part0 -> kinematic_base
- joint baselink_to_part0: origin xyz=0 0 0.95 rpy=3.14 0 3.14 -> xyz=0 0 0.95 rpy=0 0 3.141592654
