Commit message: part0 rotation fixed

File: uwsim/data/scenes/g500ARM5.urdf.xacro (robot description, xacro)
@@ -24,5 +24,5 @@
   <link name="part0">
     <visual>
-      <origin rpy="0.0 0 0" xyz="0 0 0"/>
+      <origin rpy="${pi} 0 0" xyz="0 0 0"/>
       <geometry>
         <mesh filename="${robot_parts_path}_part0.${ext}"/>
